File: Hannes256.kicad_pcb (KiCad board)
At the start: 2 copper layers, 56.3 x 82 mm, 38 parts, among them J1 TED_SOCKET, J2 RAM_SELECTOR, J3 CONN_CS, U1 MOS_7360_TED, U10 41256, U11 41256, U12 41256, U13 41256, U14 41256, U15 NE555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

Commit message: Final touches
Routing:
- net /~RAS~/~CAS~ Generation/~cs_ramrd: track 42.5 -> 41.6 mm
- net GND: vias 15 -> 19
Other:
- board text added: "256kB RAM Expansion for the Commodore 16 Based on work by Hannes and Solder/Synergy Thanks to TLC!"
- board text added: "CC-BY-NC-SA © SukkoPera 2022-2023 github.com/ SukkoPera/ Hannes256"
- board text removed: "256kB RAM Expansion for the Commodore 16 Based on work by Hannes and Solder/Synergy"
- board text removed: "CC-BY-NC-SA © SukkoPera 2022 github.com/ SukkoPera/ Hannes256"
Changed lines of the file:
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@@
     (thickness 1.6)
     (drawings 26)
-    (tracks 1183)
+    (tracks 1185)
     (zones 0)
     (modules 38)
@@
   (title_block
     (title Hannes256)
-    (date 2023-01-09)
+    (date 2023-03-14)
     (rev 3git)
     (company SukkoPera)
@@
     (tags "capacitor handsolder")
     (attr smd)
-    (fp_text reference C3 (at 2.667 0 90) (layer F.SilkS)
+    (fp_text reference C3 (at -2.4645 0 90) (layer F.SilkS)
       (effects (font (size 1 1) (thickness 0.15)))
     )
@@
     (tags "resistor array")
     (attr smd)
-    (fp_text reference RN1 (at 2.921 0 270) (layer F.SilkS)
+    (fp_text reference RN1 (at -2.032 0 90) (layer F.SilkS)
       (effects (font (size 1 1) (thickness 0.15)))
     )
@@
     (tags "resistor array")
     (attr smd)
-    (fp_text reference RN2 (at 2.921 0 270) (layer F.SilkS)
+    (fp_text reference RN2 (at -2.032 0 90) (layer F.SilkS)
       (effects (font (size 1 1) (thickness 0.15)))
     )
@@
     (tags "capacitor handsolder")
     (attr smd)
-    (fp_text reference C4 (at -2.667 0 270) (layer F.SilkS)
+    (fp_text reference C4 (at -2.5915 0 270) (layer F.SilkS)
       (effects (font (size 1 1) (thickness 0.15)))
     )
@@
     (tags "SO SO")
     (attr smd)
-    (fp_text reference U3 (at 5.461 -4.318 90) (layer F.SilkS)
+    (fp_text reference U3 (at 5.3975 -4.445 90) (layer F.SilkS)
       (effects (font (size 1 1) (thickness 0.15)))
     )
@@
     (tags "SO SO")
     (attr smd)
-    (fp_text reference U4 (at -5.334 -4.445 90) (layer F.SilkS)
+    (fp_text reference U4 (at -5.3975 -4.445 90) (layer F.SilkS)
       (effects (font (size 1 1) (thickness 0.15)))
     )
@@
     )
   )
-  (gr_text "CC-BY-NC-SA\n© SukkoPera 2022\n\ngithub.com/\nSukkoPera/\nHannes256" (at 126.5195 135.166 90) (layer B.SilkS)
+  (gr_text "CC-BY-NC-SA\n© SukkoPera 2022-2023\n\ngithub.com/\nSukkoPera/\nHannes256" (at 126.5195 135.166 90) (layer B.SilkS)
     (effects (font (size 0.9 0.9) (thickness 0.15)) (justify right mirror))
   )
-  (gr_text "256kB RAM Expansion for the Commodore 16\nBased on work by Hannes and Solder/Synergy" (at 109.9245 110.231 90) (layer B.SilkS)
+  (gr_text "256kB RAM Expansion for the Commodore 16\nBased on work by Hannes and Solder/Synergy\nThanks to TLC!" (at 109.9245 110.231 90) (layer B.SilkS)
     (effects (font (size 1 1) (thickness 0.15)) (justify mirror))
   )
@@
   (via (at 132.715 68.326) (size 0.8) (drill 0.6) (layers F.Cu B.Cu) (net 18))
   (via (at 129.1575 136.652) (size 0.8) (drill 0.6) (layers F.Cu B.Cu) (net 18))
+  (via (at 110.108999 81.661) (size 0.6) (drill 0.4) (layers F.Cu B.Cu) (net 18))
+  (via (at 111.506 83.566) (size 0.6) (drill 0.4) (layers F.Cu B.Cu) (net 18))
+  (via (at 110.108999 76.581) (size 0.6) (drill 0.4) (layers F.Cu B.Cu) (net 18))
+  (via (at 110.108999 70.231) (size 0.6) (drill 0.4) (layers F.Cu B.Cu) (net 18))
   (segment (start 135.89 111.506) (end 137.414 109.982) (width 0.18) (layer B.Cu) (net 19) (status 10))
   (segment (start 137.414 109.982) (end 137.414 92.456) (width 0.18) (layer B.Cu) (net 19))
@@
   (segment (start 108.077 84.836) (end 106.6465 84.836) (width 0.18) (layer F.Cu) (net 45) (status 20))
   (segment (start 108.077 77.216) (end 106.6465 77.216) (width 0.18) (layer F.Cu) (net 45) (status 20))
-  (segment (start 115.951 78.486) (end 117.475 78.486) (width 0.18) (layer F.Cu) (net 45) (status 20))
+  (segment (start 115.951 78.486) (end 117.475 78.486) (width 0.18) (layer F.Cu) (net 45))
+  (segment (start 110.49 79.121) (end 115.316 79.121) (width 0.18) (layer F.Cu) (net 45))
   (segment (start 115.316 79.121) (end 115.951 78.486) (width 0.18) (layer F.Cu) (net 45))
-  (segment (start 111.9505 79.121) (end 115.316 79.121) (width 0.18) (layer F.Cu) (net 45))
-  (segment (start 110.74549 77.91599) (end 111.9505 79.121) (width 0.18) (layer F.Cu) (net 45))
-  (segment (start 108.77699 77.91599) (end 110.74549 77.91599) (width 0.18) (layer F.Cu) (net 45))
+  (segment (start 109.28499 77.91599) (end 110.49 79.121) (width 0.18) (layer F.Cu) (net 45))
+  (segment (start 108.77699 77.91599) (end 109.28499 77.91599) (width 0.18) (layer F.Cu) (net 45))
   (segment (start 108.077 77.216) (end 108.77699 77.91599) (width 0.18) (layer F.Cu) (net 45))
   (segment (start 132.715 136.906) (end 135.89 136.906) (width 0.18) (layer F.Cu) (net 46) (status 30))
@@
   (segment (start 112.141 98.425) (end 112.141 101.981) (width 0.18) (layer B.Cu) (net 71))
   (segment (start 108.077 101.981) (end 112.141 101.981) (width 0.18) (layer F.Cu) (net 71))
-  (via (at 109.982 78.486) (size 0.6) (drill 0.4) (layers F.Cu B.Cu) (net 72))
-  (segment (start 109.982 78.486) (end 106.6465 78.486) (width 0.18) (layer F.Cu) (net 72))
   (via (at 109.601 114.046) (size 0.6) (drill 0.4) (layers F.Cu B.Cu) (net 72))
   (segment (start 106.172 114.046) (end 109.601 114.046) (width 0.18) (layer F.Cu) (net 72))
-  (segment (start 109.982 78.486) (end 109.982 85.725) (width 0.18) (layer B.Cu) (net 72))
-  (segment (start 109.982 85.725) (end 109.601 86.106) (width 0.18) (layer B.Cu) (net 72))
   (segment (start 109.601 86.106) (end 109.601 114.046) (width 0.18) (layer B.Cu) (net 72))
+  (segment (start 109.601 86.106) (end 109.601 83.058) (width 0.18) (layer B.Cu) (net 72))
+  (segment (start 109.601 83.058) (end 108.966 82.423) (width 0.18) (layer B.Cu) (net 72))
+  (segment (start 108.966 82.423) (end 108.966 78.486) (width 0.18) (layer B.Cu) (net 72))
+  (segment (start 108.966 78.486) (end 106.6465 78.486) (width 0.18) (layer F.Cu) (net 72))
+  (via (at 108.966 78.486) (size 0.6) (drill 0.4) (layers F.Cu B.Cu) (net 72))
   (via (at 108.966 100.076) (size 0.6) (drill 0.4) (layers F.Cu B.Cu) (net 73))
   (segment (start 121.412 100.076) (end 108.966 100.076) (width 0.18) (layer F.Cu) (net 73))
@@
   (segment (start 106.172 121.666) (end 108.966 121.666) (width 0.18) (layer F.Cu) (net 73))
   (via (at 108.966 121.666) (size 0.6) (drill 0.4) (layers F.Cu B.Cu) (net 73))
-  (segment (start 109.34701 85.47099) (end 109.347 85.471) (width 0.18) (layer B.Cu) (net 74))
-  (via (at 109.347 85.471) (size 0.6) (drill 0.4) (layers F.Cu B.Cu) (net 74))
-  (segment (start 109.347 84.201) (end 109.347 85.471) (width 0.18) (layer F.Cu) (net 74))
-  (segment (start 108.712 83.566) (end 109.347 84.201) (width 0.18) (layer F.Cu) (net 74))
-  (segment (start 108.712 83.566) (end 106.6465 83.566) (width 0.18) (layer F.Cu) (net 74) (status 20))
   (segment (start 123.2325 102.616) (end 124.2075 102.616) (width 0.18) (layer F.Cu) (net 74))
   (segment (start 122.682 102.0655) (end 123.2325 102.616) (width 0.18) (layer F.Cu) (net 74))
@@
   (segment (start 122.682 98.806) (end 122.682 102.0655) (width 0.18) (layer F.Cu) (net 74))
   (segment (start 114.681 95.631) (end 116.504999 97.454999) (width 0.18) (layer F.Cu) (net 74))
-  (segment (start 108.966 85.852) (end 109.347 85.471) (width 0.18) (layer B.Cu) (net 74))
   (segment (start 108.966 95.631) (end 108.966 85.852) (width 0.18) (layer B.Cu) (net 74))
   (segment (start 108.966 95.631) (end 114.681 95.631) (width 0.18) (layer F.Cu) (net 74))
   (via (at 108.966 95.631) (size 0.6) (drill 0.4) (layers F.Cu B.Cu) (net 74))
+  (via (at 108.966 83.566) (size 0.6) (drill 0.4) (layers F.Cu B.Cu) (net 74))
+  (segment (start 108.966 85.852) (end 108.966 83.566) (width 0.18) (layer B.Cu) (net 74))
+  (segment (start 108.966 83.566) (end 106.6465 83.566) (width 0.18) (layer F.Cu) (net 74))
   (segment (start 127 102.997) (end 127.889 103.886) (width 0.18) (layer F.Cu) (net 76))
   (segment (start 126.746 96.52) (end 126.746 98.425) (width 0.18) (layer F.Cu) (net 76))
