File: Hannes256.sch (KiCad schematic (older format))
At the start: 7 parts, among them J1 TED_SOCKET, J2 RAM_SELECTOR, J3 CONN_CS, U1 MOS_7360_TED

Commit message: Add P/Ns
Parts:
- R1, R2: LCSC (none) -> C17414
- U1, V0: LCSC (none) -> -; MouserPN (none) -> -
Changed lines of the file:
@@
 F 2 "Package_DIP:DIP-48_W15.24mm_Socket_LongPads" H 6250 4135 50  0001 C CNN
 F 3 "DOCUMENTATION" H 6250 4135 50  0001 C CNN
+F 4 "-" H 6250 4135 50  0001 C CNN "LCSC"
+F 5 "-" H 6250 4135 50  0001 C CNN "MouserPN"
 	1    6250 4135
 	1    0    0    -1
@@
 F 2 "Resistor_SMD:R_0805_2012Metric_Pad1.20x1.40mm_HandSolder" V 11975 3445 50  0001 C CNN
 F 3 "~" H 12045 3445 50  0001 C CNN
+F 4 "C17414" H 12045 3445 50  0001 C CNN "LCSC"
 	1    12045 3445
 	1    0    0    -1
@@
 F 2 "Resistor_SMD:R_0805_2012Metric_Pad1.20x1.40mm_HandSolder" V 11685 3445 50  0001 C CNN
 F 3 "~" H 11755 3445 50  0001 C CNN
+F 4 "C17414" H 11755 3445 50  0001 C CNN "LCSC"
 	1    11755 3445
 	1    0    0    -1
@@
 F 2 "Hannes256:cc_by_nc_sa" H 15540 9765 50  0001 C CNN
 F 3 "" H 15540 9765 50  0001 C CNN
+F 4 "-" H 15540 9765 50  0001 C CNN "LCSC"
+F 5 "-" H 15540 9765 50  0001 C CNN "MouserPN"
 	1    15540 9765
 	1    0    0    -1
