File: ram.sch (KiCad schematic (older format))
At the start: 16 parts, among them U10 41256, U11 41256, U12 41256, U13 41256, U14 41256, U7 41256, U8 41256, U9 41256

Commit message: Add P/Ns
Parts:
- C10, C11, C12, C13, C14, C7, C8, C9: LCSC (none) -> C49678
- U10, U11, U12, U13, U14, U7, U8, U9: Notes (none) -> See README for supported chips
Changed lines of the file:
@@
 F 2 "Package_DIP:DIP-16_W7.62mm_Socket" H 4790 2525 50  0001 C CNN
 F 3 "DOCUMENTATION" H 4790 2525 50  0001 C CNN
+F 4 "See README for supported chips" H 4790 2525 50  0001 C CNN "Notes"
 	1    4790 2525
 	1    0    0    -1
@@
 F 2 "Package_DIP:DIP-16_W7.62mm_Socket" H 4790 7145 50  0001 C CNN
 F 3 "DOCUMENTATION" H 4790 7145 50  0001 C CNN
+F 4 "See README for supported chips" H 4790 7145 50  0001 C CNN "Notes"
 	1    4790 7145
 	1    0    0    -1
@@
 F 2 "Package_DIP:DIP-16_W7.62mm_Socket" H 9515 2525 50  0001 C CNN
 F 3 "DOCUMENTATION" H 9515 2525 50  0001 C CNN
+F 4 "See README for supported chips" H 9515 2525 50  0001 C CNN "Notes"
 	1    9515 2525
 	1    0    0    -1
@@
 F 2 "Package_DIP:DIP-16_W7.62mm_Socket" H 9515 4045 50  0001 C CNN
 F 3 "DOCUMENTATION" H 9515 4045 50  0001 C CNN
+F 4 "See README for supported chips" H 9515 4045 50  0001 C CNN "Notes"
 	1    9515 4045
 	1    0    0    -1
@@
 F 2 "Package_DIP:DIP-16_W7.62mm_Socket" H 9515 5625 50  0001 C CNN
 F 3 "DOCUMENTATION" H 9515 5625 50  0001 C CNN
+F 4 "See README for supported chips" H 9515 5625 50  0001 C CNN "Notes"
 	1    9515 5625
 	1    0    0    -1
@@
 F 2 "Package_DIP:DIP-16_W7.62mm_Socket" H 9515 7145 50  0001 C CNN
 F 3 "DOCUMENTATION" H 9515 7145 50  0001 C CNN
+F 4 "See README for supported chips" H 9515 7145 50  0001 C CNN "Notes"
 	1    9515 7145
 	1    0    0    -1
@@
 F 2 "Package_DIP:DIP-16_W7.62mm_Socket" H 4790 4045 50  0001 C CNN
 F 3 "DOCUMENTATION" H 4790 4045 50  0001 C CNN
+F 4 "See README for supported chips" H 4790 4045 50  0001 C CNN "Notes"
 	1    4790 4045
 	1    0    0    -1
@@
 F 2 "Package_DIP:DIP-16_W7.62mm_Socket" H 4790 5625 50  0001 C CNN
 F 3 "DOCUMENTATION" H 4790 5625 50  0001 C CNN
+F 4 "See README for supported chips" H 4790 5625 50  0001 C CNN "Notes"
 	1    4790 5625
 	1    0    0    -1
@@
 F 2 "Capacitor_SMD:C_0805_2012Metric_Pad1.18x1.45mm_HandSolder" H 6438 2420 50  0001 C CNN
 F 3 "~" H 6400 2570 50  0001 C CNN
+F 4 "C49678" H 6400 2570 50  0001 C CNN "LCSC"
 	1    6400 2570
 	1    0    0    -1
@@
 F 2 "Capacitor_SMD:C_0805_2012Metric_Pad1.18x1.45mm_HandSolder" H 6438 3940 50  0001 C CNN
 F 3 "~" H 6400 4090 50  0001 C CNN
+F 4 "C49678" H 6400 4090 50  0001 C CNN "LCSC"
 	1    6400 4090
 	1    0    0    -1
@@
 F 2 "Capacitor_SMD:C_0805_2012Metric_Pad1.18x1.45mm_HandSolder" H 6438 5520 50  0001 C CNN
 F 3 "~" H 6400 5670 50  0001 C CNN
+F 4 "C49678" H 6400 5670 50  0001 C CNN "LCSC"
 	1    6400 5670
 	1    0    0    -1
@@
 F 2 "Capacitor_SMD:C_0805_2012Metric_Pad1.18x1.45mm_HandSolder" H 6438 7050 50  0001 C CNN
 F 3 "~" H 6400 7200 50  0001 C CNN
+F 4 "C49678" H 6400 7200 50  0001 C CNN "LCSC"
 	1    6400 7200
 	1    0    0    -1
@@
 F 2 "Capacitor_SMD:C_0805_2012Metric_Pad1.18x1.45mm_HandSolder" H 11048 2420 50  0001 C CNN
 F 3 "~" H 11010 2570 50  0001 C CNN
+F 4 "C49678" H 11010 2570 50  0001 C CNN "LCSC"
 	1    11010 2570
 	1    0    0    -1
@@
 F 2 "Capacitor_SMD:C_0805_2012Metric_Pad1.18x1.45mm_HandSolder" H 11048 3940 50  0001 C CNN
 F 3 "~" H 11010 4090 50  0001 C CNN
+F 4 "C49678" H 11010 4090 50  0001 C CNN "LCSC"
 	1    11010 4090
 	1    0    0    -1
@@
 F 2 "Capacitor_SMD:C_0805_2012Metric_Pad1.18x1.45mm_HandSolder" H 11048 5520 50  0001 C CNN
 F 3 "~" H 11010 5670 50  0001 C CNN
+F 4 "C49678" H 11010 5670 50  0001 C CNN "LCSC"
 	1    11010 5670
 	1    0    0    -1
@@
 F 2 "Capacitor_SMD:C_0805_2012Metric_Pad1.18x1.45mm_HandSolder" H 11048 7050 50  0001 C CNN
 F 3 "~" H 11010 7200 50  0001 C CNN
+F 4 "C49678" H 11010 7200 50  0001 C CNN "LCSC"
 	1    11010 7200
 	1    0    0    -1
