File: ras_cas_gen.sch (KiCad schematic (older format))
At the start: 10 parts, among them U2 GAL20V8, U3 74HCT74, U4 74HCT74, U5 74HCT257, U6 74HCT257

Commit message: Bring R/W to the GAL We'll have to write an essay on this...
Connections:
- net labels added: R_~W
- wire segments 135 -> 138
- no-connect marks 8 -> 7
Other:
- note added: "R/~W~ WAS NOT USED BY THE ORIGINAL\nHANNES/SOLDER CIRCUIT. WE ADDED IT\nIN ORDER TO AVOID A GLITCH WHENEVER\nA REGISTER WRITE IS PERFORMED, SINCE\nAPPARENTLY EVERY WRITE IS ALWAYS\nPRECEDED BY A READ, WHICH MIGHT\nTRIGGER THE TEMPORARY STORING OF A\nWRONG VALUE IN OUR REGISTERS.\n(SEE WIKI)"
- moved on the sheet: C5, C6, U5, U6

Commit message: Add a 74x245 to provide RAM register read functionality
Parts:
- added U15: 74LS245, Package_SO:SOIC-20W_7.5x12.8mm_P1.27mm, symbol 74xx:74LS245
Connections:
- net labels added: d2, d3, d4, d5, ~cs_ramrd, ~cs_ramwr
- net labels removed: ~cs_ram
- wire segments 138 -> 164
- no-connect marks 7 -> 6
Other:
- note added: "... AND WE EVEN NEED SOMETHING ELSE TO LET\nOUR RAM CONTROL REGISTER TO BE READ BACK :("
- note added: "GAL22V10 CAN BE\nUSED AS WELL"
- note added: "THE 6529B IS HARD TO FIND THESE DAYS, SO A REPLACEMENT\nSHOULD BE FOUND. MANY CHIPS SEEM SUITABLE BUT THEY ALL\nLACK THE ABILITY TO PRESET THEIR OUTPUTS TO HIGH. THE\n74XX74 IS THE ONLY COMMON CHIP THAT EASILY ALLOWS THIS,\nSO WE WENT FOR IT. UNFORTUNATELY WE'LL NEED TWO..."
- note removed: "THE 6529B IS HARD TO FIND THESE DAYS, SO A REPLACEMENT\nSHOULD BE FOUND. MANY CHIPS SEEM SUITABLE BUT THEY ALL\nLACK THE ABILITY TO PRESET THEIR OUTPUTS TO HIGH. THE\n74XX74 IS THE ONLY COMMON CHIP THAT EASILY ALLOWS THIS,\nSO WE WENT FOR IT. UNFORTUNATELY WE'LL NEED TWO."
Changed lines of the file:
@@
 $EndDescr
 Text Label 7490 2960 2    50   ~ 0
-~cs_ram
+~cs_ramwr
 Text Notes 7515 2955 0    50   ~ 0
 FD16 (RAM)
@@
 	3105 10405 3105 10605
 Text Notes 5370 8345 0    50   ~ 0
-THE 6529B IS HARD TO FIND THESE DAYS, SO A REPLACEMENT\nSHOULD BE FOUND. MANY CHIPS SEEM SUITABLE BUT THEY ALL\nLACK THE ABILITY TO PRESET THEIR OUTPUTS TO HIGH. THE\n74XX74 IS THE ONLY COMMON CHIP THAT EASILY ALLOWS THIS,\nSO WE WENT FOR IT. UNFORTUNATELY WE'LL NEED TWO.
+THE 6529B IS HARD TO FIND THESE DAYS, SO A REPLACEMENT\nSHOULD BE FOUND. MANY CHIPS SEEM SUITABLE BUT THEY ALL\nLACK THE ABILITY TO PRESET THEIR OUTPUTS TO HIGH. THE\n74XX74 IS THE ONLY COMMON CHIP THAT EASILY ALLOWS THIS,\nSO WE WENT FOR IT. UNFORTUNATELY WE'LL NEED TWO...
 Wire Wire Line
 	5495 3660 5605 3660
@@
 Entry Wire Line
 	13035 5755 12935 5855
-NoConn ~ 7105 3260
 NoConn ~ 7105 3360
 Wire Wire Line
@@
 Text Notes 7475 2660 0    50   ~ 0
 R/~W~ WAS NOT USED BY THE ORIGINAL\nHANNES/SOLDER CIRCUIT. WE ADDED IT\nIN ORDER TO AVOID A GLITCH WHENEVER\nA REGISTER WRITE IS PERFORMED, SINCE\nAPPARENTLY EVERY WRITE IS ALWAYS\nPRECEDED BY A READ, WHICH MIGHT\nTRIGGER THE TEMPORARY STORING OF A\nWRONG VALUE IN OUR REGISTERS.\n(SEE WIKI)
+$Comp
+L 74xx:74LS245 U15
+U 1 1 6366E91A
+P 11575 7495
+F 0 "U15" H 11805 8145 50  0000 C CNN
+F 1 "74LS245" H 11815 6835 50  0000 C CNN
+F 2 "Package_SO:SOIC-20W_7.5x12.8mm_P1.27mm" H 11575 7495 50  0001 C CNN
+F 3 "http://www.ti.com/lit/gpn/sn74LS245" H 11575 7495 50  0001 C CNN
+	1    11575 7495
+	1    0    0    -1
+$EndComp
+Text Label 10810 7695 0    50   ~ 0
+d7
+Entry Wire Line
+	10710 7795 10810 7695
+Wire Bus Line
+	10710 7795 10180 7795
+Text GLabel 10180 7795 0    50   Input ~ 0
+d[0..7]
+Wire Wire Line
+	10810 7695 11075 7695
+Wire Wire Line
+	11075 6995 10810 6995
+Wire Wire Line
+	11075 7095 10810 7095
+Wire Wire Line
+	11075 7195 10810 7195
+Wire Wire Line
+	11075 7295 10810 7295
+Wire Wire Line
+	11075 7395 10810 7395
+Wire Wire Line
+	11075 7495 10810 7495
+Wire Wire Line
+	11075 7595 10810 7595
+Text Label 10810 6995 0    50   ~ 0
+d0
+Text Label 10810 7095 0    50   ~ 0
+d1
+Text Label 10810 7195 0    50   ~ 0
+d2
+Text Label 10810 7295 0    50   ~ 0
+d3
+Text Label 10810 7395 0    50   ~ 0
+d4
+Text Label 10810 7495 0    50   ~ 0
+d5
+Text Label 10810 7595 0    50   ~ 0
+d6
+Entry Wire Line
+	10710 7195 10810 7095
+Entry Wire Line
+	10710 7295 10810 7195
+Entry Wire Line
+	10710 7395 10810 7295
+Entry Wire Line
+	10710 7495 10810 7395
+Entry Wire Line
+	10710 7595 10810 7495
+Entry Wire Line
+	10710 7695 10810 7595
+Entry Wire Line
+	10710 7095 10810 6995
+Wire Wire Line
+	12075 6995 12305 6995
+Wire Wire Line
+	12075 7095 12305 7095
+Wire Wire Line
+	12075 7595 12305 7595
+Wire Wire Line
+	12075 7695 12305 7695
+Text Label 12305 6995 2    50   ~ 0
+p0
+Text Label 12305 7095 2    50   ~ 0
+p1
+Text Label 12305 7595 2    50   ~ 0
+p6
+Text Label 12305 7695 2    50   ~ 0
+p7
+Wire Wire Line
+	12075 7195 12160 7195
+Wire Wire Line
+	11575 8295 11575 8380
+Wire Wire Line
+	11575 6610 11575 6695
+$Comp
+L power:+5V #PWR?
+U 1 1 637951AE
+P 11575 6610
+AR Path="/637951AE" Ref="#PWR?"  Part="1"
+AR Path="/62E48B71/637951AE" Ref="#PWR?"  Part="1"
+AR Path="/63A22C28/637951AE" Ref="#PWR0112"  Part="1"
+F 0 "#PWR0112" H 11575 6460 50  0001 C CNN
+F 1 "+5V" H 11590 6783 50  0000 C CNN
+F 2 "" H 11575 6610 50  0001 C CNN
+F 3 "" H 11575 6610 50  0001 C CNN
+	1    11575 6610
+	1    0    0    -1
+$EndComp
+$Comp
+L power:+5V #PWR?
+U 1 1 63795939
+P 12160 6610
+AR Path="/63795939" Ref="#PWR?"  Part="1"
+AR Path="/62E48B71/63795939" Ref="#PWR?"  Part="1"
+AR Path="/63A22C28/63795939" Ref="#PWR0113"  Part="1"
+F 0 "#PWR0113" H 12160 6460 50  0001 C CNN
+F 1 "+5V" H 12175 6783 50  0000 C CNN
+F 2 "" H 12160 6610 50  0001 C CNN
+F 3 "" H 12160 6610 50  0001 C CNN
+	1    12160 6610
+	1    0    0    -1
+$EndComp
+$Comp
+L power:GND #PWR?
+U 1 1 63795E43
+P 11575 8380
+AR Path="/63795E43" Ref="#PWR?"  Part="1"
+AR Path="/62E48B71/63795E43" Ref="#PWR?"  Part="1"
+AR Path="/63A22C28/63795E43" Ref="#PWR0114"  Part="1"
+F 0 "#PWR0114" H 11575 8130 50  0001 C CNN
+F 1 "GND" H 11580 8207 50  0000 C CNN
+F 2 "" H 11575 8380 50  0001 C CNN
+F 3 "" H 11575 8380 50  0001 C CNN
+	1    11575 8380
+	1    0    0    -1
+$EndComp
+Wire Wire Line
+	7105 3260 7490 3260
+Text Label 7490 3260 2    50   ~ 0
+~cs_ramrd
+Text Label 10560 7995 0    50   ~ 0
+~cs_ramrd
+Wire Wire Line
+	11075 7995 10560 7995
+Wire Wire Line
+	11075 7895 10980 7895
+Wire Wire Line
+	10980 7895 10980 8285
+$Comp
+L power:GND #PWR?
+U 1 1 637AE754
+P 10980 8285
+AR Path="/637AE754" Ref="#PWR?"  Part="1"
+AR Path="/62E48B71/637AE754" Ref="#PWR?"  Part="1"
+AR Path="/63A22C28/637AE754" Ref="#PWR0115"  Part="1"
+F 0 "#PWR0115" H 10980 8035 50  0001 C CNN
+F 1 "GND" H 10985 8112 50  0000 C CNN
+F 2 "" H 10980 8285 50  0001 C CNN
+F 3 "" H 10980 8285 50  0001 C CNN
+	1    10980 8285
+	1    0    0    -1
+$EndComp
+Text Notes 10630 8870 0    50   ~ 0
+... AND WE EVEN NEED SOMETHING ELSE TO LET\nOUR RAM CONTROL REGISTER TO BE READ BACK :(
+Wire Wire Line
+	12075 7295 12160 7295
+Wire Wire Line
+	12160 6610 12160 7195
+Connection ~ 12160 7195
+Wire Wire Line
+	12160 7195 12160 7295
+Wire Wire Line
+	12075 7395 12160 7395
+Wire Wire Line
+	12160 7395 12160 7295
+Connection ~ 12160 7295
+Wire Wire Line
+	12075 7495 12160 7495
+Wire Wire Line
+	12160 7495 12160 7395
+Connection ~ 12160 7395
 Wire Bus Line
 	5420 5535 5420 7340
+Wire Bus Line
+	10710 7095 10710 7795
 Wire Bus Line
 	5090 2250 5090 3455
@@
 Wire Bus Line
 	10285 2250 10285 4950
+Text Notes 6085 2300 0    50   ~ 0
+GAL22V10 CAN BE\nUSED AS WELL
 $EndSCHEMATC

Commit message: Use a different MOS 6529 replacement circuit, courtesy of TLC
Parts:
- removed U15: 74LS245, Package_SO:SOIC-20W_7.5x12.8mm_P1.27mm, symbol 74xx:74LS245
- removed U3, U4: 74HCT74, Package_SO:SOIC-14_3.9x8.7mm_P1.27mm, symbol 74xx:74LS74
- added C15: 100n, Capacitor_SMD:C_0805_2012Metric_Pad1.18x1.45mm_HandSolder, symbol Device:C
- added C16: 10n, Capacitor_SMD:C_0805_2012Metric_Pad1.18x1.45mm_HandSolder, symbol Device:C
- added RN1, RN2: 1k, Resistor_SMD:R_Array_Convex_4x0603, symbol Device:R_Pack04
- added U15: NE555D, Package_SO:SOIC-8_3.9x4.9mm_P1.27mm, symbol Timer:NE555D
- added U3: 74LS573, Package_SO:SOIC-20W_7.5x12.8mm_P1.27mm, symbol 74xx:74LS573
- added U4: 74LS245, Package_SO:SOIC-20W_7.5x12.8mm_P1.27mm, symbol 74xx:74LS245
Connections:
- net labels added: p2, p3, p4, p5, p[0..7], ~p~[0..7], ~u3enable
- wire segments 164 -> 165
- no-connect marks 6 -> 3
Other:
- note added: "$FD16 READ"
- note added: "$FD16 WRITE"
- note added: "BISTABLE CONFIGURATION"
- note added: "INTERMEDIATE SIGNAL TO WORKAROUND\nGAL LIMITATIONS - LEAVE UNCONNECTED"
- note added: "R/~W~ WAS NOT USED IN THE ORIGINAL\nHANNES/SOLDER CIRCUIT BUT WE NEED IT\nIN ORDER TO KNOW WHETHER TO ENABLE\nTHE 74x74 OR THE 74x245."
- note added: "THE 6529B IS HARD TO FIND THESE DAYS, SO A REPLACEMENT\nSHOULD BE FOUND. MANY CHIPS SEEM SUITABLE BUT THEY ALL\nLACK THE ABILITY TO PRESET THEIR OUTPUTS TO HIGH, WHICH\nIS ESSENTIAL FOR HOW THIS EXPANSION WORKS, SO WE MUST\nRESORT TO SOME TRICK...\n\nTHERE IS NO NEED FOR OPEN-COLLECTOR OUTPUTS."
- note added: "WE ALSO NEED SOMETHING ELSE TO ALLOW OUR\nRAM CONTROL REGISTER TO BE READ BACK. SINCE\nWE ARE WORKING WITH REVERSE LOGIC, WE USE\nAN INVERTING BUFFER AND... TA-DA!"
- note added: "~RESET"
- note added: "~SET"
- note removed: "... AND WE EVEN NEED SOMETHING ELSE TO LET\nOUR RAM CONTROL REGISTER TO BE READ BACK :("
- note removed: "FD16 (RAM)"
- note removed: "R/~W~ WAS NOT USED BY THE ORIGINAL\nHANNES/SOLDER CIRCUIT. WE ADDED IT\nIN ORDER TO AVOID A GLITCH WHENEVER\nA REGISTER WRITE IS PERFORMED, SINCE\nAPPARENTLY EVERY WRITE IS ALWAYS\nPRECEDED BY A READ, WHICH MIGHT\nTRIGGER THE TEMPORARY STORING OF A\nWRONG VALUE IN OUR REGISTERS.\n(SEE WIKI)"
- note removed: "THE 6529B IS HARD TO FIND THESE DAYS, SO A REPLACEMENT\nSHOULD BE FOUND. MANY CHIPS SEEM SUITABLE BUT THEY ALL\nLACK THE ABILITY TO PRESET THEIR OUTPUTS TO HIGH. THE\n74XX74 IS THE ONLY COMMON CHIP THAT EASILY ALLOWS THIS,\nSO WE WENT FOR IT. UNFORTUNATELY WE'LL NEED TWO..."
- moved on the sheet: C3

Commit message: Update silkscreen
Parts:
- U15: value NE555D -> NE555
- U3: value 74LS573 -> 74HCT573; MouserPN (none) -> 595-SN74HCT573NSR
- U4: value 74LS245 -> 74HCT245; MouserPN (none) -> 595-SN74HCT245ANSR
Changed lines of the file:
@@
 P 6055 6265
 F 0 "U3" H 6255 6915 50  0000 C CNN
-F 1 "74LS573" H 6315 5585 50  0000 C CNN
+F 1 "74HCT573" H 6315 5585 50  0000 C CNN
 F 2 "Package_SO:SOIC-20W_7.5x12.8mm_P1.27mm" H 6055 6265 50  0001 C CNN
 F 3 "74xx/74hc573.pdf" H 6055 6265 50  0001 C CNN
+F 4 "595-SN74HCT573NSR" H 6055 6265 50  0001 C CNN "MouserPN"
 	1    6055 6265
 	1    0    0    -1
@@
 P 3520 7350
 F 0 "U15" H 3770 7705 50  0000 C CNN
-F 1 "NE555D" H 3735 6990 50  0000 C CNN
+F 1 "NE555" H 3735 6990 50  0000 C CNN
 F 2 "Package_SO:SOIC-8_3.9x4.9mm_P1.27mm" H 4370 6950 50  0001 C CNN
 F 3 "http://www.ti.com/lit/ds/symlink/ne555.pdf" H 4370 6950 50  0001 C CNN
@@
 P 11575 7495
 F 0 "U4" H 11790 8140 50  0000 C CNN
-F 1 "74LS245" H 11800 6830 50  0000 C CNN
+F 1 "74HCT245" H 11800 6830 50  0000 C CNN
 F 2 "Package_SO:SOIC-20W_7.5x12.8mm_P1.27mm" H 11575 7495 50  0001 C CNN
 F 3 "http://www.ti.com/lit/gpn/sn74LS245" H 11575 7495 50  0001 C CNN
+F 4 "595-SN74HCT245ANSR" H 11575 7495 50  0001 C CNN "MouserPN"
 	1    11575 7495
 	1    0    0    -1

Commit message: Fix U3 Latch Enable, sigh... GAL equations TBD
Connections:
- net ~cs_ramwr: no longer U3.11 (Load)
- net cs_ramwr: now reaches U2.18 (O3)
- net cs_ramwr: now also U3.11 (Load)
- no-connect marks 3 -> 2
Changed lines of the file:
@@
 Sheet 3 3
 Title "Hannes256: C16/+4 256 kB RAM Expansion"
-Date "2022-12-04"
+Date "2023-01-09"
 Rev "2git"
 Comp "SukkoPera"
@@
 Entry Wire Line
 	13035 5755 12935 5855
-NoConn ~ 7105 3360
 Wire Wire Line
 	7105 3160 9570 3160
@@
 $EndComp
 Text Label 5095 6665 0    50   ~ 0
-~cs_ramwr
+cs_ramwr
 Wire Wire Line
 	5090 5765 5555 5765
@@
 Text Label 7490 2960 2    50   ~ 0
 ~cs_ramwr
+Wire Wire Line
+	7105 3360 7490 3360
+Text Label 7490 3360 2    50   ~ 0
+cs_ramwr
 Wire Bus Line
 	7590 3760 7590 4535

Commit message: Use narrower footprint for U3/U4 and move everything on the top layer
Parts:
- U3, U4: footprint Package_SO:SOIC-20W_7.5x12.8mm_P1.27mm -> Package_SO:SO-20_5.3x12.6mm_P1.27mm
Changed lines of the file:
@@
 F 0 "U3" H 6255 6915 50  0000 C CNN
 F 1 "74HCT573" H 6315 5585 50  0000 C CNN
-F 2 "Package_SO:SOIC-20W_7.5x12.8mm_P1.27mm" H 6055 6265 50  0001 C CNN
+F 2 "Package_SO:SO-20_5.3x12.6mm_P1.27mm" H 6055 6265 50  0001 C CNN
 F 3 "74xx/74hc573.pdf" H 6055 6265 50  0001 C CNN
 F 4 "595-SN74HCT573NSR" H 6055 6265 50  0001 C CNN "MouserPN"
@@
 F 0 "U4" H 11790 8140 50  0000 C CNN
 F 1 "74HCT245" H 11800 6830 50  0000 C CNN
-F 2 "Package_SO:SOIC-20W_7.5x12.8mm_P1.27mm" H 11575 7495 50  0001 C CNN
+F 2 "Package_SO:SO-20_5.3x12.6mm_P1.27mm" H 11575 7495 50  0001 C CNN
 F 3 "http://www.ti.com/lit/gpn/sn74LS245" H 11575 7495 50  0001 C CNN
 F 4 "595-SN74HCT245ANSR" H 11575 7495 50  0001 C CNN "MouserPN"

Commit message: Add P/Ns
Parts:
- C15, C2, C3, C4, C5, C6: LCSC (none) -> C49678
- C16: LCSC (none) -> C1710
- RN1, RN2: LCSC (none) -> C20197
- U15: LCSC (none) -> C5125085
- U3: LCSC (none) -> C2864941
- U4: LCSC (none) -> C133641
- U5, U6: LCSC (none) -> C707097; Notes (none) -> HCT recommended, '157 works just as well
Changed lines of the file:
@@
 F 2 "Capacitor_SMD:C_0805_2012Metric_Pad1.18x1.45mm_HandSolder" H 4453 3060 50  0001 C CNN
 F 3 "~" H 4415 3210 50  0001 C CNN
+F 4 "C49678" H 4415 3210 50  0001 C CNN "LCSC"
 	1    4415 3210
 	1    0    0    -1
@@
 F 2 "Package_SO:SOIC-16_3.9x9.9mm_P1.27mm" H 11735 4750 50  0001 C CNN
 F 3 "" H 11735 4750 50  0001 C CNN
+F 4 "C707097" H 11735 4750 50  0001 C CNN "LCSC"
+F 5 "HCT recommended, '157 works just as well" H 11735 4750 50  0001 C CNN "Notes"
 	1    11735 4750
 	1    0    0    -1
@@
 F 2 "Package_SO:SOIC-16_3.9x9.9mm_P1.27mm" H 11735 3050 50  0001 C CNN
 F 3 "" H 11735 3050 50  0001 C CNN
+F 4 "C707097" H 11735 3050 50  0001 C CNN "LCSC"
+F 5 "HCT recommended, '157 works just as well" H 11735 3050 50  0001 C CNN "Notes"
 	1    11735 3050
 	1    0    0    -1
@@
 F 2 "Capacitor_SMD:C_0805_2012Metric_Pad1.18x1.45mm_HandSolder" H 13523 4505 50  0001 C CNN
 F 3 "~" H 13485 4655 50  0001 C CNN
+F 4 "C49678" H 13485 4655 50  0001 C CNN "LCSC"
 	1    13485 4655
 	1    0    0    -1
@@
 F 2 "Capacitor_SMD:C_0805_2012Metric_Pad1.18x1.45mm_HandSolder" H 13523 2870 50  0001 C CNN
 F 3 "~" H 13485 3020 50  0001 C CNN
+F 4 "C49678" H 13485 3020 50  0001 C CNN "LCSC"
 	1    13485 3020
 	1    0    0    -1
@@
 F 2 "Capacitor_SMD:C_0805_2012Metric_Pad1.18x1.45mm_HandSolder" H 4628 5635 50  0001 C CNN
 F 3 "~" H 4590 5785 50  0001 C CNN
+F 4 "C49678" H 4590 5785 50  0001 C CNN "LCSC"
 	1    4590 5785
 	1    0    0    -1
@@
 F 3 "74xx/74hc573.pdf" H 6055 6265 50  0001 C CNN
 F 4 "595-SN74HCT573NSR" H 6055 6265 50  0001 C CNN "MouserPN"
+F 5 "C2864941" H 6055 6265 50  0001 C CNN "LCSC"
 	1    6055 6265
 	1    0    0    -1
@@
 F 2 "Package_SO:SOIC-8_3.9x4.9mm_P1.27mm" H 4370 6950 50  0001 C CNN
 F 3 "http://www.ti.com/lit/ds/symlink/ne555.pdf" H 4370 6950 50  0001 C CNN
+F 4 "C5125085" H 3520 7350 50  0001 C CNN "LCSC"
 	1    3520 7350
 	1    0    0    -1
@@
 F 2 "Capacitor_SMD:C_0805_2012Metric_Pad1.18x1.45mm_HandSolder" H 2943 7675 50  0001 C CNN
 F 3 "~" H 2905 7825 50  0001 C CNN
+F 4 "C1710" H 2905 7825 50  0001 C CNN "LCSC"
 	1    2905 7825
 	1    0    0    -1
@@
 F 2 "Resistor_SMD:R_Array_Convex_4x0603" V 7035 5425 50  0001 C CNN
 F 3 "~" H 6760 5425 50  0001 C CNN
+F 4 "C20197" H 6760 5425 50  0001 C CNN "LCSC"
 	1    6760 5425
 	-1   0    0    -1
@@
 F 2 "Resistor_SMD:R_Array_Convex_4x0603" V 7650 5425 50  0001 C CNN
 F 3 "~" H 7375 5425 50  0001 C CNN
+F 4 "C20197" H 7375 5425 50  0001 C CNN "LCSC"
 	1    7375 5425
 	-1   0    0    -1
@@
 F 3 "http://www.ti.com/lit/gpn/sn74LS245" H 11575 7495 50  0001 C CNN
 F 4 "595-SN74HCT245ANSR" H 11575 7495 50  0001 C CNN "MouserPN"
+F 5 "C133641" H 11575 7495 50  0001 C CNN "LCSC"
 	1    11575 7495
 	1    0    0    -1
@@
 F 2 "Capacitor_SMD:C_0805_2012Metric_Pad1.18x1.45mm_HandSolder" H 13068 6825 50  0001 C CNN
 F 3 "~" H 13030 6975 50  0001 C CNN
+F 4 "C49678" H 13030 6975 50  0001 C CNN "LCSC"
 	1    13030 6975
 	1    0    0    -1
@@
 F 2 "Capacitor_SMD:C_0805_2012Metric_Pad1.18x1.45mm_HandSolder" H 2188 7175 50  0001 C CNN
 F 3 "~" H 2150 7325 50  0001 C CNN
+F 4 "C49678" H 2150 7325 50  0001 C CNN "LCSC"
 	1    2150 7325
 	1    0    0    -1
